File: KP08_keypad/KP08_keypad.kicad_pcb (KiCad board)
At the start: 2 copper layers, 97.8 x 39.4 mm, 21 parts, among them J1 Conn_01x13, J2 Conn_01x13, J3 Conn_01x03, SW1 SW_Push, SW10 SW_Push_SPDT, SW11 SW_Push, SW12 SW_Push_SPDT, SW2 SW_Push, SW3 SW_Push, SW4 SW_Push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

Commit message: Update footprint
Parts:
- moved SW10 1.05 mm to (94.0, 69.4)
- moved SW12 1.05 mm to (94.0, 69.4)
- moved REF** 0.25 mm to (161.9, 68.3)
- moved REF** 0.25 mm to (123.8, 68.3)
- moved REF** 0.25 mm to (161.9, 103.1)
Routing:
- net GND: track 242.6 -> 63.5 mm, vias 2 -> 4
- net Net-(J3-Pad2): track 11.9 -> 14.0 mm
- net KEY_8: track 120.1 -> 118.3 mm
- net +BATT: track 19.8 -> 18.3 mm
- net RESET: track 32.8 -> 32.2 mm

Commit message: Change mount hole from M3 to M2
Parts:
- removed the REF** at (161.9, 103.1)
- removed the REF** at (161.9, 68.3)
- removed the REF** at (123.8, 85.7)
- removed the REF** at (161.9, 85.7)
- removed the REF** at (123.8, 68.3)
- added REF**: MountingHole_2.2mm_M2, MountingHole:MountingHole_2.2mm_M2, F.Cu at (161.9, 85.7)
- added REF**: MountingHole_2.2mm_M2, MountingHole:MountingHole_2.2mm_M2, F.Cu at (161.9, 103.5)
- added REF**: MountingHole_2.2mm_M2, MountingHole:MountingHole_2.2mm_M2, F.Cu at (161.9, 67.9)
- added REF**: MountingHole_2.2mm_M2, MountingHole:MountingHole_2.2mm_M2, F.Cu at (123.8, 85.7)
- added REF**: MountingHole_2.2mm_M2, MountingHole:MountingHole_2.2mm_M2, F.Cu at (123.8, 67.9)
- REF**: value MountingHole_3.2mm_M3 -> MountingHole_2.2mm_M2; footprint MountingHole:MountingHole_3.2mm_M3 -> MountingHole:MountingHole_2.2mm_M2
- moved REF** 1.27 mm to (94.0, 91.4)
